File: arena_w_vreg/teensy_arena_12-12/teensy_arena_12-12_tmp.kicad_pcb (KiCad board)
At the start: 4 copper layers, 254 x 254 mm, 87 parts, among them J1 Barrel_Jack, J2 Conn_01x04, J3 Conn_01x04, P1 CONN15, P10 CONN15, P11 CONN15, P12 CONN15, P2 CONN15, P3 CONN15, P4 CONN15, P5 CONN15, P6 CONN15, P7 CONN15, P8 CONN15, P9 CONN15, Q2 MOSFET_NCHAN, SW1 SW_SPDT, U1 TXB0108PW, U10 AZ1084-5.0, U11 AZ1084-5.0, U12 AZ1084-5.0, U13 AZ1084-5.0, U14 AZ1084-5.0, U15 AZ1084-5.0, U16 AZ1084-5.0, U17 AZ1084-5.0, U18 Teensy4.1, U2 TXB0108PW, U3 TXB0108PW, U4 TXB0108PW, U5 TXB0108PW, U6 AZ1084-5.0, U7 AZ1084-5.0, U8 AZ1084-5.0, U9 AZ1084-5.0

Commit message: Worked on routing 12-12 arena with vreg.
Connections:
- P1 pad 3: /Panel Headers/RESET -> /Level Shifters/PAN5V.SCK_1
- P10 pad 3: /Panel Headers/RESET -> /Level Shifters/PAN5V.SCK_1
- P11 pad 3: /Panel Headers/RESET -> /Level Shifters/PAN5V.SCK_1
- P12 pad 3: /Panel Headers/RESET -> /Level Shifters/PAN5V.SCK_1
- P2 pad 3: /Panel Headers/RESET -> /Level Shifters/PAN5V.SCK_1
- P3 pad 3: /Panel Headers/RESET -> /Level Shifters/PAN5V.SCK_1
- P4 pad 3: /Panel Headers/RESET -> /Level Shifters/PAN5V.SCK_1
- P5 pad 3: /Panel Headers/RESET -> /Level Shifters/PAN5V.SCK_1
- P6 pad 3: /Panel Headers/RESET -> /Level Shifters/PAN5V.SCK_1
- P7 pad 3: /Panel Headers/RESET -> /Level Shifters/PAN5V.SCK_1
- P8 pad 3: /Panel Headers/RESET -> /Level Shifters/PAN5V.SCK_1
- P9 pad 3: /Panel Headers/RESET -> /Level Shifters/PAN5V.SCK_1
- Q2 pad 3: /Panel Headers/RESET -> /Level Shifters/PAN5V.SCK_1
Routing:
- net /Level Shifters/PAN5V.SCK_1: track 0.00 -> 619.6 mm, vias 0 -> 1
- net /Level Shifters/PAN5V.EXT_INT: track 0.00 -> 580.3 mm, vias 0 -> 3
- net /Level Shifters/PAN5V.CS_22: track 0.00 -> 434.5 mm, vias 0 -> 6
- net /Level Shifters/PAN5V.CS_00: track 0.00 -> 406.9 mm, vias 0 -> 3
- net /Level Shifters/PAN5V.CS_17: track 0.00 -> 402.6 mm
- net /Level Shifters/PAN5V.CS_18: track 0.00 -> 400.9 mm, vias 0 -> 3
- net /Level Shifters/PAN5V.CS_16: track 0.00 -> 399.7 mm, vias 0 -> 3
- net /Level Shifters/PAN5V.CS_19: track 0.00 -> 399.6 mm, vias 0 -> 1
- net /Level Shifters/PAN5V.CS_01: track 0.00 -> 385.1 mm, vias 0 -> 4
- net /Level Shifters/PAN5V.CS_04: track 0.00 -> 381.3 mm, vias 0 -> 4
- net /Level Shifters/PAN5V.CS_06: track 0.00 -> 364.3 mm, vias 0 -> 6
- net /Level Shifters/PAN5V.CS_29: track 0.00 -> 362.9 mm, vias 0 -> 3
- net /Level Shifters/PAN5V.CS_20: track 0.00 -> 360.0 mm, vias 0 -> 4
- net /Level Shifters/PAN5V.CS_03: track 0.00 -> 359.7 mm, vias 0 -> 3
- net /Level Shifters/PAN5V.CS_08: track 0.00 -> 359.3 mm, vias 0 -> 4
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