File: development/arena_12-12/ni/ni_arena_12-12_v0p1/panel_headers.kicad_sch (KiCad schematic)
At the start: 27 parts, among them P1 CONN15, P10 CONN15, P11 CONN15, P12 CONN15, P2 CONN15, P3 CONN15, P4 CONN15, P5 CONN15, P6 CONN15, P7 CONN15, P8 CONN15, P9 CONN15, Q2 MOSFET_NCHAN

Commit message: Further work on 12-12 ni arena.
Connections:
- net PAN5V.CS_00: now also P2.7
- net PAN5V.CS_01: now also P2.8
- net PAN5V.CS_02: now also P2.9
- net PAN5V.CS_03: now also P2.10
- net PAN5V.CS_04: now also P2.11
- net PAN5V.CS_05: now also P1.12; no longer P2.7
- net PAN5V.CS_06: now also P1.13; no longer P2.8
- net PAN5V.CS_07: now also P1.14; no longer P2.9
- net PAN5V.CS_08: no longer P2.10
- net PAN5V.CS_09: no longer P2.11
- net PAN5V.MISO_0: no longer P1.6, P2.6
- net PAN5V.MOSI_0: no longer P1.5, P2.5
- net PAN5V.SCK_0: no longer P1.4, P2.4
- new net PAN5V.MISO_00: P1.6
- new net PAN5V.MISO_01: P2.6
- new net PAN5V.MOSI_00: P1.5
- new net PAN5V.MOSI_01: P2.5
- new net PAN5V.SCK_00: P1.4
- new net PAN5V.SCK_01: P2.4
- no-connect marks 36 -> 0

Commit message: Finished initial schematic and layout for 12-12 NI arena (without voltage regulators).
Connections:
- net PAN5V.CS_08 is gone; now on net PAN5V.CS_03: P8.10
- net PAN5V.CS_09 is gone; now on net PAN5V.CS_04: P8.11
- net PAN5V.CS_10 is gone; now on net PAN5V.CS_00: P3.7, P9.7
- net PAN5V.CS_11 is gone; now on net PAN5V.CS_01: P3.8, P9.8
- net PAN5V.CS_12 is gone; now on net PAN5V.CS_02: P3.9, P9.9
- net PAN5V.CS_13 is gone; now on net PAN5V.CS_03: P3.10, P9.10
- net PAN5V.CS_14 is gone; now on net PAN5V.CS_04: P3.11, P9.11
- net PAN5V.CS_15 is gone; now on net PAN5V.CS_00: P10.7, P4.7
- net PAN5V.CS_16 is gone; now on net PAN5V.CS_01: P10.8, P4.8
- net PAN5V.CS_17 is gone; now on net PAN5V.CS_02: P10.9, P4.9
- net PAN5V.CS_18 is gone; now on net PAN5V.CS_03: P10.10, P4.10
- net PAN5V.CS_19 is gone; now on net PAN5V.CS_04: P10.11, P4.11
- net PAN5V.CS_20 is gone; now on net PAN5V.CS_00: P11.7, P5.7
- net PAN5V.CS_21 is gone; now on net PAN5V.CS_01: P11.8, P5.8
- net PAN5V.CS_22 is gone; now on net PAN5V.CS_02: P11.9, P5.9
- net PAN5V.CS_23 is gone; now on net PAN5V.CS_03: P11.10, P5.10
- net PAN5V.CS_24 is gone; now on net PAN5V.CS_04: P11.11, P5.11
- net PAN5V.CS_25 is gone; now on net PAN5V.CS_00: P12.7, P6.7
- net PAN5V.CS_26 is gone; now on net PAN5V.CS_01: P12.8, P6.8
- net PAN5V.CS_27 is gone; now on net PAN5V.CS_02: P12.9, P6.9
- net PAN5V.CS_28 is gone; now on net PAN5V.CS_03: P12.10, P6.10
- net PAN5V.CS_29 is gone; now on net PAN5V.CS_04: P12.11, P6.11
- net PAN5V.CS_00: now also P8.7
- net PAN5V.CS_01: now also P8.8
- net PAN5V.CS_02: now also P8.9
- net PAN5V.CS_05: now also P10.12, P11.12, P12.12, P2.12, P3.12, P4.12, P5.12, P6.12, P7.12, P8.12, P9.12; no longer P8.7
- net PAN5V.CS_06: now also P10.13, P11.13, P12.13, P2.13, P3.13, P4.13, P5.13, P6.13, P7.13, P8.13, P9.13; no longer P8.8
- net PAN5V.CS_07: now also P10.14, P11.14, P12.14, P2.14, P3.14, P4.14, P5.14, P6.14, P7.14, P8.14, P9.14; no longer P8.9
- net PAN5V.SCK_00: now also P7.4
- net PAN5V.SCK_01: now also P8.4
- removed net PAN5V.MISO_0: P3.6, P4.6, P5.6, P6.6
- removed net PAN5V.MISO_1: P10.6, P11.6, P12.6, P7.6, P8.6, P9.6
- removed net PAN5V.MOSI_0: P3.5, P4.5, P5.5, P6.5
- removed net PAN5V.MOSI_1: P10.5, P11.5, P12.5, P7.5, P8.5, P9.5
- removed net PAN5V.SCK_0: P3.4, P4.4, P5.4, P6.4
- removed net PAN5V.SCK_1: P10.4, P11.4, P12.4, P7.4, P8.4, P9.4
- new net PAN5V.MISO_02: P3.6
- new net PAN5V.MISO_03: P4.6
- new net PAN5V.MISO_04: P5.6
- new net PAN5V.MISO_05: P6.6
- new net PAN5V.MISO_06: P7.6
- new net PAN5V.MISO_07: P8.6
- new net PAN5V.MISO_08: P9.6
- new net PAN5V.MISO_09: P10.6
- new net PAN5V.MISO_10: P11.6
- new net PAN5V.MISO_11: P12.6
- new net PAN5V.MOSI_02: P3.5
- new net PAN5V.MOSI_03: P4.5
- new net PAN5V.MOSI_04: P5.5
- new net PAN5V.MOSI_05: P6.5
- new net PAN5V.MOSI_06: P7.5
- new net PAN5V.MOSI_07: P8.5
- new net PAN5V.MOSI_08: P9.5
- new net PAN5V.MOSI_09: P10.5
- new net PAN5V.MOSI_10: P11.5
- new net PAN5V.MOSI_11: P12.5
- new net PAN5V.SCK_02: P3.4, P9.4
- new net PAN5V.SCK_03: P10.4, P4.4
- new net PAN5V.SCK_04: P11.4, P5.4
- new net PAN5V.SCK_05: P12.4, P6.4
