File: development/arena_12-12/ni/ni_arena_12-12_v0p1/ni_arena_12-12.kicad_sch (KiCad schematic)
At the start: 0 parts

Commit message: Worked on layout for 12-12 NI arena w/ vreg.
Other:
- note added: "12-12 NI Arena"
- note removed: "12-12 Teensy Arena"
Changed lines of the file:
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@@
     (stroke (width 0) (type default))
   )
-  (text "12-12 Teensy Arena" (at 113.03 33.02 0)
-    (effects (font (size 2.54 2.54)) (justify left bottom))
+  (text "12-12 NI Arena" (at 113.03 33.02 0)
+    (effects (font (size 2.54 2.54) (thickness 0.508) bold) (justify left bottom))
   )
   (sheet (at 94.107 49.784) (size 33.147 18.034) (fields_autoplaced)
