File: development/arena_12-12/ni/ni_arena_12-12_v0p1/layout_tool/modified_ni_arena_12-12.kicad_pcb (KiCad board)
At the start: 4 copper layers, 228.6 x 228.6 mm, 51 parts, among them J1 Barrel_Jack, J2 Conn_01x04, J3 Conn_01x04, P1 CONN15, P10 CONN15, P11 CONN15, P12 CONN15, P2 CONN15, P3 CONN15, P4 CONN15, P5 CONN15, P6 CONN15, P7 CONN15, P8 CONN15, P9 CONN15, Q2 MOSFET_NCHAN, SW1 SW_SPDT, U1 TXB0108PW, U18 Teensy4.1, U2 TXB0108PW, U3 TXB0108PW, U4 TXB0108PW, U5 TXB0108PW

Commit message: Worked on 12-12 arenas.
Resized 12-12 arenas,   changed NI connector from right angle to
vertical, push panals back by 1mm.
Parts:
- removed J3: Conn_01x04, arena_custom:JST_SH_SM04B-SRSS-TB_1x04-1MP_P1.00mm_Horizontal
- removed U18: Teensy4.1, teensy:Teensy41
- added C23: 10uF, Capacitor_SMD:C_0603_1608Metric, F.Cu at (299.7, 131.5)
- added C24: 10uF, Capacitor_SMD:C_0603_1608Metric, F.Cu at (296.2, 135.8)
- added H5: MountingHole_Pad, MountingHole:MountingHole_4.5mm_Pad, F.Cu at (292.1, 190.5)
- added H6: MountingHole_Pad, MountingHole:MountingHole_4.5mm_Pad, F.Cu at (292.1, 266.7)
- added U6: AP2112K-3.3, Package_TO_SOT_SMD:SOT-23-5, F.Cu at (296.3, 132.8)
- J2: value Conn_01x04 -> NI_TE_68pos; footprint arena_custom:JST_SH_SM04B-SRSS-TB_1x04-1MP_P1.00mm_Horizontal -> arena_custom:TE_CONN_DSUB_RA_68
- moved C2 201.8 mm to (108.1, 294.4), turned to 180 degrees
- moved C1 197.3 mm to (120.6, 294.4), turned to 0 degrees
- moved U1 196.1 mm to (114.3, 292.1), turned to 180 degrees
- moved C4 150.7 mm to (146.2, 294.4), turned to 180 degrees
- moved C3 144.3 mm to (158.4, 294.4), turned to 0 degrees
- moved U2 144.2 mm to (152.4, 292.1), turned to 180 degrees
- moved U4 106.7 mm to (266.7, 292.1)
- moved C7 106.6 mm to (272.9, 294.7)
- moved C8 106.5 mm to (260.4, 294.4)
- moved C9 78.3 mm to (196.7, 294.3)
- moved U5 78.1 mm to (190.5, 292.1)
- moved C10 77.9 mm to (184.1, 294.4)
- moved J2 68.1 mm to (304.6, 228.6)
- moved SW1 29.5 mm to (299.5, 86.2)
- moved J1 27.3 mm to (304.6, 116.5)
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Connections:
- J2 pad 2: +3.3V -> GND
- J2 pad 3: /Teensy/SDA -> GND
- J2 pad 4: /Teensy/SCL -> unconnected-(J2-Pin_4-Pad4)
- P1 pad 12: unconnected-(P1-Pad12) -> /Level Shifters/PAN5V.CS_05
- P1 pad 13: unconnected-(P1-Pad13) -> /Level Shifters/PAN5V.CS_06
- P1 pad 14: unconnected-(P1-Pad14) -> /Level Shifters/PAN5V.CS_07
- P1 pad 4: /Level Shifters/PAN5V.SCK_0 -> /Level Shifters/PAN5V.SCK_00
- P1 pad 5: /Level Shifters/PAN5V.MOSI_0 -> /Level Shifters/PAN5V.MOSI_00
- P1 pad 6: /Level Shifters/PAN5V.MISO_0 -> /Level Shifters/PAN5V.MISO_00
- P10 pad 10: /Level Shifters/PAN5V.CS_18 -> /Level Shifters/PAN5V.CS_03
- P10 pad 11: /Level Shifters/PAN5V.CS_19 -> /Level Shifters/PAN5V.CS_04
- P10 pad 12: unconnected-(P10-Pad12) -> /Level Shifters/PAN5V.CS_05
- P10 pad 13: unconnected-(P10-Pad13) -> /Level Shifters/PAN5V.CS_06
- P10 pad 14: unconnected-(P10-Pad14) -> /Level Shifters/PAN5V.CS_07
- P10 pad 4: /Level Shifters/PAN5V.SCK_1 -> /Level Shifters/PAN5V.SCK_03
- P10 pad 5: /Level Shifters/PAN5V.MOSI_1 -> /Level Shifters/PAN5V.MOSI_09
- P10 pad 6: /Level Shifters/PAN5V.MISO_1 -> /Level Shifters/PAN5V.MISO_09
- P10 pad 7: /Level Shifters/PAN5V.CS_15 -> /Level Shifters/PAN5V.CS_00
- P10 pad 8: /Level Shifters/PAN5V.CS_16 -> /Level Shifters/PAN5V.CS_01
- P10 pad 9: /Level Shifters/PAN5V.CS_17 -> /Level Shifters/PAN5V.CS_02
- P11 pad 10: /Level Shifters/PAN5V.CS_23 -> /Level Shifters/PAN5V.CS_03
- P11 pad 11: /Level Shifters/PAN5V.CS_24 -> /Level Shifters/PAN5V.CS_04
- P11 pad 12: unconnected-(P11-Pad12) -> /Level Shifters/PAN5V.CS_05
- P11 pad 13: unconnected-(P11-Pad13) -> /Level Shifters/PAN5V.CS_06
- P11 pad 14: unconnected-(P11-Pad14) -> /Level Shifters/PAN5V.CS_07
- P11 pad 4: /Level Shifters/PAN5V.SCK_1 -> /Level Shifters/PAN5V.SCK_04
- P11 pad 5: /Level Shifters/PAN5V.MOSI_1 -> /Level Shifters/PAN5V.MOSI_10
- P11 pad 6: /Level Shifters/PAN5V.MISO_1 -> /Level Shifters/PAN5V.MISO_10
- P11 pad 7: /Level Shifters/PAN5V.CS_20 -> /Level Shifters/PAN5V.CS_00
- P11 pad 8: /Level Shifters/PAN5V.CS_21 -> /Level Shifters/PAN5V.CS_01
- P11 pad 9: /Level Shifters/PAN5V.CS_22 -> /Level Shifters/PAN5V.CS_02
- P12 pad 10: /Level Shifters/PAN5V.CS_28 -> /Level Shifters/PAN5V.CS_03
- P12 pad 11: /Level Shifters/PAN5V.CS_29 -> /Level Shifters/PAN5V.CS_04
- P12 pad 12: unconnected-(P12-Pad12) -> /Level Shifters/PAN5V.CS_05
- P12 pad 13: unconnected-(P12-Pad13) -> /Level Shifters/PAN5V.CS_06
- P12 pad 14: unconnected-(P12-Pad14) -> /Level Shifters/PAN5V.CS_07
- P12 pad 4: /Level Shifters/PAN5V.SCK_1 -> /Level Shifters/PAN5V.SCK_05
- P12 pad 5: /Level Shifters/PAN5V.MOSI_1 -> /Level Shifters/PAN5V.MOSI_11
- P12 pad 6: /Level Shifters/PAN5V.MISO_1 -> /Level Shifters/PAN5V.MISO_11
- P12 pad 7: /Level Shifters/PAN5V.CS_25 -> /Level Shifters/PAN5V.CS_00
- P12 pad 8: /Level Shifters/PAN5V.CS_26 -> /Level Shifters/PAN5V.CS_01
- P12 pad 9: /Level Shifters/PAN5V.CS_27 -> /Level Shifters/PAN5V.CS_02
- P2 pad 10: /Level Shifters/PAN5V.CS_08 -> /Level Shifters/PAN5V.CS_03
- P2 pad 11: /Level Shifters/PAN5V.CS_09 -> /Level Shifters/PAN5V.CS_04
- P2 pad 12: unconnected-(P2-Pad12) -> /Level Shifters/PAN5V.CS_05
- P2 pad 13: unconnected-(P2-Pad13) -> /Level Shifters/PAN5V.CS_06
- P2 pad 14: unconnected-(P2-Pad14) -> /Level Shifters/PAN5V.CS_07
- P2 pad 4: /Level Shifters/PAN5V.SCK_0 -> /Level Shifters/PAN5V.SCK_01
- P2 pad 5: /Level Shifters/PAN5V.MOSI_0 -> /Level Shifters/PAN5V.MOSI_01
- P2 pad 6: /Level Shifters/PAN5V.MISO_0 -> /Level Shifters/PAN5V.MISO_01
- P2 pad 7: /Level Shifters/PAN5V.CS_05 -> /Level Shifters/PAN5V.CS_00
- P2 pad 8: /Level Shifters/PAN5V.CS_06 -> /Level Shifters/PAN5V.CS_01
- P2 pad 9: /Level Shifters/PAN5V.CS_07 -> /Level Shifters/PAN5V.CS_02
- P3 pad 10: /Level Shifters/PAN5V.CS_13 -> /Level Shifters/PAN5V.CS_03
- P3 pad 11: /Level Shifters/PAN5V.CS_14 -> /Level Shifters/PAN5V.CS_04
- P3 pad 12: unconnected-(P3-Pad12) -> /Level Shifters/PAN5V.CS_05
- P3 pad 13: unconnected-(P3-Pad13) -> /Level Shifters/PAN5V.CS_06
- P3 pad 14: unconnected-(P3-Pad14) -> /Level Shifters/PAN5V.CS_07
- P3 pad 4: /Level Shifters/PAN5V.SCK_0 -> /Level Shifters/PAN5V.SCK_02
- P3 pad 5: /Level Shifters/PAN5V.MOSI_0 -> /Level Shifters/PAN5V.MOSI_02
- P3 pad 6: /Level Shifters/PAN5V.MISO_0 -> /Level Shifters/PAN5V.MISO_02
- P3 pad 7: /Level Shifters/PAN5V.CS_10 -> /Level Shifters/PAN5V.CS_00
- P3 pad 8: /Level Shifters/PAN5V.CS_11 -> /Level Shifters/PAN5V.CS_01
- P3 pad 9: /Level Shifters/PAN5V.CS_12 -> /Level Shifters/PAN5V.CS_02
- P4 pad 10: /Level Shifters/PAN5V.CS_18 -> /Level Shifters/PAN5V.CS_03
- P4 pad 11: /Level Shifters/PAN5V.CS_19 -> /Level Shifters/PAN5V.CS_04
- P4 pad 12: unconnected-(P4-Pad12) -> /Level Shifters/PAN5V.CS_05
- P4 pad 13: unconnected-(P4-Pad13) -> /Level Shifters/PAN5V.CS_06
- P4 pad 14: unconnected-(P4-Pad14) -> /Level Shifters/PAN5V.CS_07
- P4 pad 4: /Level Shifters/PAN5V.SCK_0 -> /Level Shifters/PAN5V.SCK_03
- P4 pad 5: /Level Shifters/PAN5V.MOSI_0 -> /Level Shifters/PAN5V.MOSI_03
- P4 pad 6: /Level Shifters/PAN5V.MISO_0 -> /Level Shifters/PAN5V.MISO_03
- P4 pad 7: /Level Shifters/PAN5V.CS_15 -> /Level Shifters/PAN5V.CS_00
- P4 pad 8: /Level Shifters/PAN5V.CS_16 -> /Level Shifters/PAN5V.CS_01
- P4 pad 9: /Level Shifters/PAN5V.CS_17 -> /Level Shifters/PAN5V.CS_02
- P5 pad 10: /Level Shifters/PAN5V.CS_23 -> /Level Shifters/PAN5V.CS_03
- P5 pad 11: /Level Shifters/PAN5V.CS_24 -> /Level Shifters/PAN5V.CS_04
- P5 pad 12: unconnected-(P5-Pad12) -> /Level Shifters/PAN5V.CS_05
- P5 pad 13: unconnected-(P5-Pad13) -> /Level Shifters/PAN5V.CS_06
- P5 pad 14: unconnected-(P5-Pad14) -> /Level Shifters/PAN5V.CS_07
- P5 pad 4: /Level Shifters/PAN5V.SCK_0 -> /Level Shifters/PAN5V.SCK_04
- P5 pad 5: /Level Shifters/PAN5V.MOSI_0 -> /Level Shifters/PAN5V.MOSI_04
- P5 pad 6: /Level Shifters/PAN5V.MISO_0 -> /Level Shifters/PAN5V.MISO_04
- P5 pad 7: /Level Shifters/PAN5V.CS_20 -> /Level Shifters/PAN5V.CS_00
- P5 pad 8: /Level Shifters/PAN5V.CS_21 -> /Level Shifters/PAN5V.CS_01
- P5 pad 9: /Level Shifters/PAN5V.CS_22 -> /Level Shifters/PAN5V.CS_02
- P6 pad 10: /Level Shifters/PAN5V.CS_28 -> /Level Shifters/PAN5V.CS_03
- P6 pad 11: /Level Shifters/PAN5V.CS_29 -> /Level Shifters/PAN5V.CS_04
- P6 pad 12: unconnected-(P6-Pad12) -> /Level Shifters/PAN5V.CS_05
- P6 pad 13: unconnected-(P6-Pad13) -> /Level Shifters/PAN5V.CS_06
- P6 pad 14: unconnected-(P6-Pad14) -> /Level Shifters/PAN5V.CS_07
- P6 pad 4: /Level Shifters/PAN5V.SCK_0 -> /Level Shifters/PAN5V.SCK_05
- P6 pad 5: /Level Shifters/PAN5V.MOSI_0 -> /Level Shifters/PAN5V.MOSI_05
- P6 pad 6: /Level Shifters/PAN5V.MISO_0 -> /Level Shifters/PAN5V.MISO_05
- P6 pad 7: /Level Shifters/PAN5V.CS_25 -> /Level Shifters/PAN5V.CS_00
- P6 pad 8: /Level Shifters/PAN5V.CS_26 -> /Level Shifters/PAN5V.CS_01
- P6 pad 9: /Level Shifters/PAN5V.CS_27 -> /Level Shifters/PAN5V.CS_02
- P7 pad 12: unconnected-(P7-Pad12) -> /Level Shifters/PAN5V.CS_05
- P7 pad 13: unconnected-(P7-Pad13) -> /Level Shifters/PAN5V.CS_06
- P7 pad 14: unconnected-(P7-Pad14) -> /Level Shifters/PAN5V.CS_07
- P7 pad 4: /Level Shifters/PAN5V.SCK_1 -> /Level Shifters/PAN5V.SCK_00
- P7 pad 5: /Level Shifters/PAN5V.MOSI_1 -> /Level Shifters/PAN5V.MOSI_06
- P7 pad 6: /Level Shifters/PAN5V.MISO_1 -> /Level Shifters/PAN5V.MISO_06
- P8 pad 10: /Level Shifters/PAN5V.CS_08 -> /Level Shifters/PAN5V.CS_03
- P8 pad 11: /Level Shifters/PAN5V.CS_09 -> /Level Shifters/PAN5V.CS_04
- P8 pad 12: unconnected-(P8-Pad12) -> /Level Shifters/PAN5V.CS_05
- P8 pad 13: unconnected-(P8-Pad13) -> /Level Shifters/PAN5V.CS_06
- P8 pad 14: unconnected-(P8-Pad14) -> /Level Shifters/PAN5V.CS_07
- P8 pad 4: /Level Shifters/PAN5V.SCK_1 -> /Level Shifters/PAN5V.SCK_01
- P8 pad 5: /Level Shifters/PAN5V.MOSI_1 -> /Level Shifters/PAN5V.MOSI_07
- P8 pad 6: /Level Shifters/PAN5V.MISO_1 -> /Level Shifters/PAN5V.MISO_07
- P8 pad 7: /Level Shifters/PAN5V.CS_05 -> /Level Shifters/PAN5V.CS_00
- P8 pad 8: /Level Shifters/PAN5V.CS_06 -> /Level Shifters/PAN5V.CS_01
- P8 pad 9: /Level Shifters/PAN5V.CS_07 -> /Level Shifters/PAN5V.CS_02
- P9 pad 10: /Level Shifters/PAN5V.CS_13 -> /Level Shifters/PAN5V.CS_03
- P9 pad 11: /Level Shifters/PAN5V.CS_14 -> /Level Shifters/PAN5V.CS_04
- P9 pad 12: unconnected-(P9-Pad12) -> /Level Shifters/PAN5V.CS_05
- P9 pad 13: unconnected-(P9-Pad13) -> /Level Shifters/PAN5V.CS_06
- P9 pad 14: unconnected-(P9-Pad14) -> /Level Shifters/PAN5V.CS_07
- P9 pad 4: /Level Shifters/PAN5V.SCK_1 -> /Level Shifters/PAN5V.SCK_02
- P9 pad 5: /Level Shifters/PAN5V.MOSI_1 -> /Level Shifters/PAN5V.MOSI_08
- P9 pad 6: /Level Shifters/PAN5V.MISO_1 -> /Level Shifters/PAN5V.MISO_08
- P9 pad 7: /Level Shifters/PAN5V.CS_10 -> /Level Shifters/PAN5V.CS_00
- P9 pad 8: /Level Shifters/PAN5V.CS_11 -> /Level Shifters/PAN5V.CS_01
- P9 pad 9: /Level Shifters/PAN5V.CS_12 -> /Level Shifters/PAN5V.CS_02
- U1 pad 1: /Level Shifters/PAN3V.RESET -> /Level Shifters/PAN3V.CS_00
- U1 pad 12: /Level Shifters/PAN5V.MISO_1 -> /Level Shifters/PAN5V.CS_07
- U1 pad 13: /Level Shifters/PAN5V.MOSI_1 -> /Level Shifters/PAN5V.CS_06
- U1 pad 14: /Level Shifters/PAN5V.SCK_1 -> /Level Shifters/PAN5V.CS_05
- U1 pad 15: unconnected-(U1-B5-Pad15) -> /Level Shifters/PAN5V.CS_04
- U1 pad 16: /Level Shifters/PAN5V.MISO_0 -> /Level Shifters/PAN5V.CS_03
- U1 pad 17: /Level Shifters/PAN5V.MOSI_0 -> /Level Shifters/PAN5V.CS_02
- U1 pad 18: /Level Shifters/PAN5V.SCK_0 -> /Level Shifters/PAN5V.CS_01
- U1 pad 20: /Level Shifters/PAN5V.RESET -> /Level Shifters/PAN5V.CS_00
- U1 pad 3: /Level Shifters/PAN3V.SCK_0 -> /Level Shifters/PAN3V.CS_01
- U1 pad 4: /Level Shifters/PAN3V.MOSI_0 -> /Level Shifters/PAN3V.CS_02
- U1 pad 5: /Level Shifters/PAN3V.MISO_0 -> /Level Shifters/PAN3V.CS_03
- U1 pad 6: unconnected-(U1-A5-Pad6) -> /Level Shifters/PAN3V.CS_04
- U1 pad 7: /Level Shifters/PAN3V.SCK_1 -> /Level Shifters/PAN3V.CS_05
- U1 pad 8: /Level Shifters/PAN3V.MOSI_1 -> /Level Shifters/PAN3V.CS_06
- U1 pad 9: /Level Shifters/PAN3V.MISO_1 -> /Level Shifters/PAN3V.CS_07
- U2 pad 1: /Level Shifters/PAN3V.CS_00 -> /Level Shifters/PAN3V.SCK_00
- U2 pad 12: /Level Shifters/PAN5V.CS_07 -> /Level Shifters/PAN5V.MISO_00
- U2 pad 13: /Level Shifters/PAN5V.CS_06 -> /Level Shifters/PAN5V.MOSI_00
- U2 pad 14: /Level Shifters/PAN5V.CS_05 -> /Level Shifters/PAN5V.SCK_05
- U2 pad 15: /Level Shifters/PAN5V.CS_04 -> /Level Shifters/PAN5V.SCK_04
- U2 pad 16: /Level Shifters/PAN5V.CS_03 -> /Level Shifters/PAN5V.SCK_03
- U2 pad 17: /Level Shifters/PAN5V.CS_02 -> /Level Shifters/PAN5V.SCK_02
- U2 pad 18: /Level Shifters/PAN5V.CS_01 -> /Level Shifters/PAN5V.SCK_01
- U2 pad 20: /Level Shifters/PAN5V.CS_00 -> /Level Shifters/PAN5V.SCK_00
- U2 pad 3: /Level Shifters/PAN3V.CS_01 -> /Level Shifters/PAN3V.SCK_01
- U2 pad 4: /Level Shifters/PAN3V.CS_02 -> /Level Shifters/PAN3V.SCK_02
- U2 pad 5: /Level Shifters/PAN3V.CS_03 -> /Level Shifters/PAN3V.SCK_03
- U2 pad 6: /Level Shifters/PAN3V.CS_04 -> /Level Shifters/PAN3V.SCK_04
- U2 pad 7: /Level Shifters/PAN3V.CS_05 -> /Level Shifters/PAN3V.SCK_05
- U2 pad 8: /Level Shifters/PAN3V.CS_06 -> /Level Shifters/PAN3V.MOSI_00
- U2 pad 9: /Level Shifters/PAN3V.CS_07 -> /Level Shifters/PAN3V.MISO_00
- U3 pad 1: /Level Shifters/PAN3V.CS_08 -> /Level Shifters/PAN3V.MOSI_01
- U3 pad 12: /Level Shifters/PAN5V.CS_15 -> /Level Shifters/PAN5V.MISO_04
- U3 pad 13: /Level Shifters/PAN5V.CS_14 -> /Level Shifters/PAN5V.MOSI_04
- U3 pad 14: /Level Shifters/PAN5V.CS_13 -> /Level Shifters/PAN5V.MISO_03
- U3 pad 15: /Level Shifters/PAN5V.CS_12 -> /Level Shifters/PAN5V.MOSI_03
- U3 pad 16: /Level Shifters/PAN5V.CS_11 -> /Level Shifters/PAN5V.MISO_02
- U3 pad 17: /Level Shifters/PAN5V.CS_10 -> /Level Shifters/PAN5V.MOSI_02
- U3 pad 18: /Level Shifters/PAN5V.CS_09 -> /Level Shifters/PAN5V.MISO_01
- U3 pad 20: /Level Shifters/PAN5V.CS_08 -> /Level Shifters/PAN5V.MOSI_01
- U3 pad 3: /Level Shifters/PAN3V.CS_09 -> /Level Shifters/PAN3V.MISO_01
- U3 pad 4: /Level Shifters/PAN3V.CS_10 -> /Level Shifters/PAN3V.MOSI_02
- U3 pad 5: /Level Shifters/PAN3V.CS_11 -> /Level Shifters/PAN3V.MISO_02
- U3 pad 6: /Level Shifters/PAN3V.CS_12 -> /Level Shifters/PAN3V.MOSI_03
- U3 pad 7: /Level Shifters/PAN3V.CS_13 -> /Level Shifters/PAN3V.MISO_03
- U3 pad 8: /Level Shifters/PAN3V.CS_14 -> /Level Shifters/PAN3V.MOSI_04
- U3 pad 9: /Level Shifters/PAN3V.CS_15 -> /Level Shifters/PAN3V.MISO_04
- U4 pad 1: /Level Shifters/PAN3V.CS_16 -> /Level Shifters/PAN3V.MOSI_05
- U4 pad 12: /Level Shifters/PAN5V.CS_23 -> /Level Shifters/PAN5V.MISO_08
- U4 pad 13: /Level Shifters/PAN5V.CS_22 -> /Level Shifters/PAN5V.MOSI_08
- U4 pad 14: /Level Shifters/PAN5V.CS_21 -> /Level Shifters/PAN5V.MISO_07
- U4 pad 15: /Level Shifters/PAN5V.CS_20 -> /Level Shifters/PAN5V.MOSI_07
- U4 pad 16: /Level Shifters/PAN5V.CS_19 -> /Level Shifters/PAN5V.MISO_06
- U4 pad 17: /Level Shifters/PAN5V.CS_18 -> /Level Shifters/PAN5V.MOSI_06
- U4 pad 18: /Level Shifters/PAN5V.CS_17 -> /Level Shifters/PAN5V.MISO_05
- U4 pad 20: /Level Shifters/PAN5V.CS_16 -> /Level Shifters/PAN5V.MOSI_05
- U4 pad 3: /Level Shifters/PAN3V.CS_17 -> /Level Shifters/PAN3V.MISO_05
- U4 pad 4: /Level Shifters/PAN3V.CS_18 -> /Level Shifters/PAN3V.MOSI_06
- U4 pad 5: /Level Shifters/PAN3V.CS_19 -> /Level Shifters/PAN3V.MISO_06
- U4 pad 6: /Level Shifters/PAN3V.CS_20 -> /Level Shifters/PAN3V.MOSI_07
- U4 pad 7: /Level Shifters/PAN3V.CS_21 -> /Level Shifters/PAN3V.MISO_07
- U4 pad 8: /Level Shifters/PAN3V.CS_22 -> /Level Shifters/PAN3V.MOSI_08
- U4 pad 9: /Level Shifters/PAN3V.CS_23 -> /Level Shifters/PAN3V.MISO_08
- U5 pad 1: /Level Shifters/PAN3V.CS_24 -> /Level Shifters/PAN3V.MOSI_09
- U5 pad 12: /Level Shifters/PAN5V.EXT_INT -> /Level Shifters/PAN5V.RESET
- U5 pad 13: unconnected-(U5-B7-Pad13) -> /Level Shifters/PAN5V.EXT_INT
- U5 pad 14: /Level Shifters/PAN5V.CS_29 -> /Level Shifters/PAN5V.MISO_11
- U5 pad 15: /Level Shifters/PAN5V.CS_28 -> /Level Shifters/PAN5V.MOSI_11
- U5 pad 16: /Level Shifters/PAN5V.CS_27 -> /Level Shifters/PAN5V.MISO_10
- U5 pad 17: /Level Shifters/PAN5V.CS_26 -> /Level Shifters/PAN5V.MOSI_10
- U5 pad 18: /Level Shifters/PAN5V.CS_25 -> /Level Shifters/PAN5V.MISO_09
- U5 pad 20: /Level Shifters/PAN5V.CS_24 -> /Level Shifters/PAN5V.MOSI_09
- U5 pad 3: /Level Shifters/PAN3V.CS_25 -> /Level Shifters/PAN3V.MISO_09
- U5 pad 4: /Level Shifters/PAN3V.CS_26 -> /Level Shifters/PAN3V.MOSI_10
- U5 pad 5: /Level Shifters/PAN3V.CS_27 -> /Level Shifters/PAN3V.MISO_10
- U5 pad 6: /Level Shifters/PAN3V.CS_28 -> /Level Shifters/PAN3V.MOSI_11
- U5 pad 7: /Level Shifters/PAN3V.CS_29 -> /Level Shifters/PAN3V.MISO_11
- U5 pad 8: unconnected-(U5-A7-Pad8) -> /Level Shifters/PAN3V.EXT_INT
- U5 pad 9: /Level Shifters/PAN3V.EXT_INT -> /Level Shifters/PAN3V.RESET
Other:
- outline, holes or cut-outs redrawn
- board text added: "NI 12-12 Arena V0.1 R1"
- board text removed: "Teensy 12-12 Controller-Arena V0.1 R1"
