File: development/arena_12-12/teensy4p1/teensy_arena_12-12_v0p1/layout_tool/modified_teensy_arena_12-12.kicad_pcb (KiCad board)
At the start: 4 copper layers, 228.6 x 228.6 mm, 51 parts, among them J1 Barrel_Jack, J2 Conn_01x04, J3 Conn_01x04, P1 CONN15, P10 CONN15, P11 CONN15, P12 CONN15, P2 CONN15, P3 CONN15, P4 CONN15, P5 CONN15, P6 CONN15, P7 CONN15, P8 CONN15, P9 CONN15, Q2 MOSFET_NCHAN, SW1 SW_SPDT, U1 TXB0108PW, U18 Teensy4.1, U2 TXB0108PW, U3 TXB0108PW, U4 TXB0108PW, U5 TXB0108PW

Commit message: Worked on 12-12 arenas.
Resized 12-12 arenas,   changed NI connector from right angle to
vertical, push panals back by 1mm.
Parts:
- moved C7 107.9 mm to (274.3, 293.6)
- moved C8 107.9 mm to (261.9, 293.7)
- moved U4 107.9 mm to (268.0, 291.4)
- moved J2 78.2 mm to (301.5, 239.5)
- moved J3 78.2 mm to (301.5, 230.5)
- moved C10 74.1 mm to (180.4, 293.6)
- moved C9 74.1 mm to (192.5, 293.6)
- moved U5 74.1 mm to (186.5, 291.3)
- moved R1 34.1 mm to (293.5, 167.6)
- moved R2 34.1 mm to (295.4, 164.3)
- moved Q2 34.1 mm to (291.5, 164.3)
- moved C1 32.5 mm to (273.9, 220.5), turned to 180 degrees
- moved SW1 29.5 mm to (299.5, 86.2)
- moved J1 27.3 mm to (304.6, 116.5)
- moved U1 24.8 mm to (280.9, 222.8), turned to 0 degrees
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Other:
- outline, holes or cut-outs redrawn
