File: development/arena_12-12_w_vreg/teensy4p1/teensy_arena_12-12_v0p2/teensy_arena_12-12.kicad_pcb (KiCad board)
At the start: 4 copper layers, 254 x 254 mm, 87 parts, among them J1 Barrel_Jack, J2 Conn_01x04, J3 Conn_01x04, P1 CONN15, P10 CONN15, P11 CONN15, P12 CONN15, P2 CONN15, P3 CONN15, P4 CONN15, P5 CONN15, P6 CONN15, P7 CONN15, P8 CONN15, P9 CONN15, Q2 MOSFET_NCHAN, SW1 SW_SPDT, U1 TXB0108PW, U10 AZ1084-5.0, U11 AZ1084-5.0, U12 AZ1084-5.0, U13 AZ1084-5.0, U14 AZ1084-5.0, U15 AZ1084-5.0, U16 AZ1084-5.0, U17 AZ1084-5.0, U18 Teensy4.1, U2 TXB0108PW, U3 TXB0108PW, U4 TXB0108PW, U5 TXB0108PW, U6 AZ1084-5.0, U7 AZ1084-5.0, U8 AZ1084-5.0, U9 AZ1084-5.0

Commit message: Added work on switching regulator.
Parts:
- added C35: 10uF, Capacitor_SMD:C_0603_1608Metric, F.Cu at (-62.0, 75.4)
- added C36: 100nF, Capacitor_SMD:C_0603_1608Metric, F.Cu at (-62.0, 77.9)
- added C37: 22uF, Capacitor_SMD:C_0603_1608Metric, F.Cu at (-62.0, 80.4)
- added C38: 10uF, Capacitor_SMD:C_0603_1608Metric, F.Cu at (-62.0, 82.9)
- added C39: 100nF, Capacitor_SMD:C_0603_1608Metric, F.Cu at (-62.0, 85.4)
- added C40: 22uF, Capacitor_SMD:C_0603_1608Metric, F.Cu at (-62.0, 87.9)
- added C41: 10uF, Capacitor_SMD:C_0603_1608Metric, F.Cu at (-62.0, 90.4)
- added C42: 100nF, Capacitor_SMD:C_0603_1608Metric, F.Cu at (-62.0, 92.9)
- added C43: 22uF, Capacitor_SMD:C_0603_1608Metric, F.Cu at (-62.0, 95.4)
- added C44: 10uF, Capacitor_SMD:C_0603_1608Metric, F.Cu at (-58.0, 70.3)
- added C45: 100nF, Capacitor_SMD:C_0603_1608Metric, F.Cu at (-58.0, 72.9)
- added C46: 22uF, Capacitor_SMD:C_0603_1608Metric, F.Cu at (-58.0, 75.4)
- added L1: 3.3uH, arena_custom:CYA0650_3P3UH, F.Cu at (274.2, 158.2)
- added L10: 3.3uH, arena_custom:CYA0650_3P3UH, F.Cu at (-40.5, 100.6)
- added L11: 3.3uH, arena_custom:CYA0650_3P3UH, F.Cu at (-40.5, 108.3)
- added L12: 3.3uH, arena_custom:CYA0650_3P3UH, F.Cu at (-39.9, 117.6)
- added L2: 3.3uH, arena_custom:CYA0650_3P3UH, F.Cu at (-67.5, 108.3)
- added L3: 3.3uH, arena_custom:CYA0650_3P3UH, F.Cu at (-67.5, 116.0)
- added L4: 3.3uH, arena_custom:CYA0650_3P3UH, F.Cu at (-58.5, 100.6)
- added L5: 3.3uH, arena_custom:CYA0650_3P3UH, F.Cu at (-58.5, 108.3)
- added L6: 3.3uH, arena_custom:CYA0650_3P3UH, F.Cu at (-58.5, 116.0)
- added L7: 3.3uH, arena_custom:CYA0650_3P3UH, F.Cu at (-49.5, 100.6)
- added L8: 3.3uH, arena_custom:CYA0650_3P3UH, F.Cu at (-49.5, 108.3)
- added L9: 3.3uH, arena_custom:CYA0650_3P3UH, F.Cu at (-49.5, 116.0)
- added R15: 56.2k, Resistor_SMD:R_0603_1608Metric, F.Cu at (-54.0, 80.4)
- added R16: 10k, Resistor_SMD:R_0603_1608Metric, F.Cu at (-54.0, 82.9)
- added R17: 56.2k, Resistor_SMD:R_0603_1608Metric, F.Cu at (-54.0, 85.4)
- added R18: 10k, Resistor_SMD:R_0603_1608Metric, F.Cu at (-54.0, 87.9)
- added R19: 56.2k, Resistor_SMD:R_0603_1608Metric, F.Cu at (-54.0, 90.4)
- added R20: 10k, Resistor_SMD:R_0603_1608Metric, F.Cu at (-54.0, 92.9)
- added R21: 56.2k, Resistor_SMD:R_0603_1608Metric, F.Cu at (-54.0, 95.4)
- added R22: 10k, Resistor_SMD:R_0603_1608Metric, F.Cu at (-50.0, 70.3)
- added R23: 56.2k, Resistor_SMD:R_0603_1608Metric, F.Cu at (-50.0, 72.9)
- added R24: 10k, Resistor_SMD:R_0603_1608Metric, F.Cu at (-50.0, 75.4)
- added R25: 56.2k, Resistor_SMD:R_0603_1608Metric, F.Cu at (-50.0, 77.9)
- added R26: 10k, Resistor_SMD:R_0603_1608Metric, F.Cu at (-50.0, 80.4)
- C11, C15, C21, C27, C33: value 10uF -> 100nF; footprint Capacitor_SMD:CP_Elec_4x5.4 -> Capacitor_SMD:C_0603_1608Metric
- C12, C14, C20, C26, C32: value 22uF -> 10uF; footprint Capacitor_SMD:CP_Elec_4x5.4 -> Capacitor_SMD:C_0603_1608Metric
- C13, C19, C25, C31: value 10uF -> 22uF; footprint Capacitor_SMD:CP_Elec_4x5.4 -> Capacitor_SMD:C_0603_1608Metric
- C16, C17, C22, C23, C28, C29, C34: footprint Capacitor_SMD:CP_Elec_4x5.4 -> Capacitor_SMD:C_0603_1608Metric
- C18, C24, C30: value 22uF -> 100nF; footprint Capacitor_SMD:CP_Elec_4x5.4 -> Capacitor_SMD:C_0603_1608Metric
- R10, R12, R14, R4, R6, R8: value 300 -> 10k; footprint Resistor_SMD:R_1206_3216Metric -> Resistor_SMD:R_0603_1608Metric
- R11, R13, R3, R5, R7, R9: value 300 -> 56.2k; footprint Resistor_SMD:R_1206_3216Metric -> Resistor_SMD:R_0603_1608Metric
- U10, U11, U12, U13, U14, U15, U16, U17, U6, U7, U8, U9: value AZ1084-5.0 -> TPS564201DDC; footprint arena_custom:TO-252 -> Package_TO_SOT_SMD:SOT-23-6
- moved C33 362.3 mm to (-62.0, 70.3), turned to 0 degrees
- moved C34 361.5 mm to (-62.0, 72.9), turned to 0 degrees
- moved R14 352.1 mm to (-54.0, 77.9), turned to 0 degrees
- moved C14 346.1 mm to (-70.0, 77.9), turned to 0 degrees
- moved R13 336.9 mm to (-54.0, 75.4), turned to 0 degrees
- moved C32 334.2 mm to (-66.0, 95.4), turned to 0 degrees
- moved U17 329.6 mm to (-30.0, 80.2), turned to 0 degrees
- moved C31 329.4 mm to (-66.0, 92.9), turned to 0 degrees
- moved U7 326.7 mm to (-45.4, 75.8), turned to 0 degrees
- moved C15 320.7 mm to (-70.0, 80.4), turned to 0 degrees
- moved U16 313.3 mm to (-30.0, 75.8), turned to 0 degrees
- moved C16 308.5 mm to (-70.0, 82.9), turned to 0 degrees
- moved R12 304.6 mm to (-54.0, 72.9), turned to 0 degrees
- moved C30 299.1 mm to (-66.0, 90.4), turned to 0 degrees
- moved R5 292.4 mm to (-58.0, 82.9), turned to 0 degrees
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Connections:
- C11 pad 1: VCC -> Net-(U6-VBST)
- C11 pad 2: GND -> Net-(U6-SW)
- C12 pad 1: /Panel Headers/POW.5V_HDR_1 -> VCC
- C13 pad 1: VCC -> GND
- C13 pad 2: GND -> /Panel Headers/POW.5V_HDR_1
- C14 pad 1: /Panel Headers/POW.5V_HDR_2 -> VCC
- C15 pad 1: VCC -> Net-(U7-VBST)
- C15 pad 2: GND -> Net-(U7-SW)
- C16 pad 1: /Panel Headers/POW.5V_HDR_3 -> GND
- C16 pad 2: GND -> /Panel Headers/POW.5V_HDR_2
- C18 pad 1: /Panel Headers/POW.5V_HDR_4 -> Net-(U8-VBST)
- C18 pad 2: GND -> Net-(U8-SW)
- C19 pad 1: VCC -> GND
- C19 pad 2: GND -> /Panel Headers/POW.5V_HDR_3
- C20 pad 1: /Panel Headers/POW.5V_HDR_5 -> VCC
- C21 pad 1: VCC -> Net-(U9-VBST)
- C21 pad 2: GND -> Net-(U9-SW)
- C22 pad 1: /Panel Headers/POW.5V_HDR_6 -> GND
- C22 pad 2: GND -> /Panel Headers/POW.5V_HDR_4
- C24 pad 1: /Panel Headers/POW.5V_HDR_7 -> Net-(U10-VBST)
- C24 pad 2: GND -> Net-(U10-SW)
- C25 pad 1: VCC -> GND
- C25 pad 2: GND -> /Panel Headers/POW.5V_HDR_5
- C26 pad 1: /Panel Headers/POW.5V_HDR_8 -> VCC
- C27 pad 1: VCC -> Net-(U11-VBST)
- C27 pad 2: GND -> Net-(U11-SW)
- C28 pad 1: /Panel Headers/POW.5V_HDR_9 -> GND
- C28 pad 2: GND -> /Panel Headers/POW.5V_HDR_6
- C30 pad 1: /Panel Headers/POW.5V_HDR_10 -> Net-(U12-VBST)
- C30 pad 2: GND -> Net-(U12-SW)
- C31 pad 1: VCC -> GND
- C31 pad 2: GND -> /Panel Headers/POW.5V_HDR_7
- C32 pad 1: /Panel Headers/POW.5V_HDR_11 -> VCC
- C33 pad 1: VCC -> Net-(U13-VBST)
- C33 pad 2: GND -> Net-(U13-SW)
- C34 pad 1: /Panel Headers/POW.5V_HDR_12 -> GND
- C34 pad 2: GND -> /Panel Headers/POW.5V_HDR_8
- R10 pad 1: /Panel Headers/POW.5V_HDR_8 -> Net-(U9-VFB)
- R11 pad 1: /Panel Headers/POW.5V_HDR_9 -> /Panel Headers/POW.5V_HDR_5
- R11 pad 2: GND -> Net-(U10-VFB)
- R12 pad 1: /Panel Headers/POW.5V_HDR_10 -> Net-(U10-VFB)
- R13 pad 1: /Panel Headers/POW.5V_HDR_11 -> /Panel Headers/POW.5V_HDR_6
- R13 pad 2: GND -> Net-(U11-VFB)
- R14 pad 1: /Panel Headers/POW.5V_HDR_12 -> Net-(U11-VFB)
- R3 pad 2: GND -> Net-(U6-VFB)
- R4 pad 1: /Panel Headers/POW.5V_HDR_2 -> Net-(U6-VFB)
- R5 pad 1: /Panel Headers/POW.5V_HDR_3 -> /Panel Headers/POW.5V_HDR_2
- R5 pad 2: GND -> Net-(U7-VFB)
- R6 pad 1: /Panel Headers/POW.5V_HDR_4 -> Net-(U7-VFB)
- R7 pad 1: /Panel Headers/POW.5V_HDR_5 -> /Panel Headers/POW.5V_HDR_3
- R7 pad 2: GND -> Net-(U8-VFB)
- R8 pad 1: /Panel Headers/POW.5V_HDR_6 -> Net-(U8-VFB)
- R9 pad 1: /Panel Headers/POW.5V_HDR_7 -> /Panel Headers/POW.5V_HDR_4
- R9 pad 2: GND -> Net-(U9-VFB)
- U10 pad 2: /Panel Headers/POW.5V_HDR_5 -> Net-(U10-SW)
- U11 pad 2: /Panel Headers/POW.5V_HDR_6 -> Net-(U11-SW)
- U12 pad 2: /Panel Headers/POW.5V_HDR_7 -> Net-(U12-SW)
- U13 pad 2: /Panel Headers/POW.5V_HDR_8 -> Net-(U13-SW)
- U14 pad 2: /Panel Headers/POW.5V_HDR_9 -> Net-(U14-SW)
- U15 pad 2: /Panel Headers/POW.5V_HDR_10 -> Net-(U15-SW)
- U16 pad 2: /Panel Headers/POW.5V_HDR_11 -> Net-(U16-SW)
- U17 pad 2: /Panel Headers/POW.5V_HDR_12 -> Net-(U17-SW)
- U6 pad 2: /Panel Headers/POW.5V_HDR_1 -> Net-(U6-SW)
- U7 pad 2: /Panel Headers/POW.5V_HDR_2 -> Net-(U7-SW)
- U8 pad 2: /Panel Headers/POW.5V_HDR_3 -> Net-(U8-SW)
- U9 pad 2: /Panel Headers/POW.5V_HDR_4 -> Net-(U9-SW)
