File: development/arena_12-12_w_vreg/teensy4p1/teensy_arena_12-12_v0p2/teensy_arena_12-12.kicad_pcb (KiCad board)
At the start: 4 copper layers, 228.6 x 228.6 mm, 123 parts, among them J1 Barrel_Jack, J2 Conn_01x04, J3 Conn_01x04, P1 CONN15, P10 CONN15, P11 CONN15, P12 CONN15, P2 CONN15, P3 CONN15, P4 CONN15, P5 CONN15, P6 CONN15, P7 CONN15, P8 CONN15, P9 CONN15, Q2 MOSFET_NCHAN, SW1 SW_SPDT, U1 TXB0108PW, U10 TPS564201DDC, U11 TPS564201DDC, U12 TPS564201DDC, U13 TPS564201DDC, U14 TPS564201DDC, U15 TPS564201DDC, U16 TPS564201DDC, U17 TPS564201DDC, U18 Teensy4.1, U2 TXB0108PW, U3 TXB0108PW, U4 TXB0108PW, U5 TXB0108PW, U6 TPS564201DDC, U7 TPS564201DDC, U8 TPS564201DDC, U9 TPS564201DDC

Commit message: Worked on layout for 12-12 NI arena w/ vreg.
Parts:
- moved U18 1.18 mm to (260.3, 270.5)
Changed lines of the file:
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@@
   )
   (footprint "teensy:Teensy41" (layer "F.Cu")
-    (at 259.366674 269.833983 -160)
+    (at 260.310378 270.545439 -160)
     (property "Sheetfile" "teensy.kicad_sch")
     (property "Sheetname" "Teensy")
