File: development/arena_12-12_w_vreg/teensy4p1/teensy_arena_12-12_v0p2/teensy_arena_12-12_backup.kicad_pcb (KiCad board)
At the start: 4 copper layers, 228.6 x 228.6 mm, 123 parts, among them J1 Barrel_Jack, J2 Conn_01x04, J3 Conn_01x04, P1 CONN15, P10 CONN15, P11 CONN15, P12 CONN15, P2 CONN15, P3 CONN15, P4 CONN15, P5 CONN15, P6 CONN15, P7 CONN15, P8 CONN15, P9 CONN15, Q2 MOSFET_NCHAN, SW1 SW_SPDT, U1 TXB0108PW, U10 TPS564201DDC, U11 TPS564201DDC, U12 TPS564201DDC, U13 TPS564201DDC, U14 TPS564201DDC, U15 TPS564201DDC, U16 TPS564201DDC, U17 TPS564201DDC, U18 Teensy4.1, U2 TXB0108PW, U3 TXB0108PW, U4 TXB0108PW, U5 TXB0108PW, U6 TPS564201DDC, U7 TPS564201DDC, U8 TPS564201DDC, U9 TPS564201DDC

Commit message: Worked on teensy41 arena w/ vreg.
Parts:
- moved C44 312.2 mm to (-9.83, 95.0), turned to 0 degrees
- moved C45 309.8 mm to (-9.83, 97.5), turned to 0 degrees
- moved C46 301.6 mm to (-9.83, 100.0), turned to 0 degrees
- moved C41 299.5 mm to (-13.8, 115.0), turned to 0 degrees
- moved R26 294.9 mm to (-1.81, 105.0), turned to 0 degrees
- moved C42 294.8 mm to (-13.8, 117.5), turned to 0 degrees
- moved R25 293.0 mm to (-1.81, 102.5), turned to 0 degrees
- moved R24 292.0 mm to (-1.81, 100.0), turned to 0 degrees
- moved C43 291.2 mm to (-13.8, 120.1), turned to 0 degrees
- moved R23 290.6 mm to (-1.81, 97.5), turned to 0 degrees
- moved C15 282.0 mm to (-21.9, 105.0), turned to 0 degrees
- moved U17 281.8 mm to (18.2, 104.8), turned to 0 degrees
- moved C14 279.8 mm to (-21.9, 102.5), turned to 0 degrees
- moved U16 278.2 mm to (18.2, 100.4), turned to 0 degrees
- moved C38 276.4 mm to (-13.8, 107.5), turned to 0 degrees
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
Commit message: Worked on routing for teensy vreg arena.
Parts:
- C11: value 100nF -> 10uF
- C12: value 10uF -> 100nF
- moved C45 310.7 mm to (279.4, 210.9), turned to 150 degrees
- moved C44 309.7 mm to (275.3, 216.0), turned to -30 degrees
- moved C46 300.9 mm to (272.8, 203.2), turned to 150 degrees
- moved C42 297.9 mm to (249.2, 257.3), turned to 120 degrees
- moved C41 294.8 mm to (243.1, 259.6), turned to -60 degrees
- moved R26 294.1 mm to (274.6, 205.4), turned to 60 degrees
- moved R25 292.2 mm to (271.9, 204.8), turned to -30 degrees
- moved R24 291.3 mm to (247.9, 250.1), turned to 30 degrees
- moved C43 290.5 mm to (247.4, 247.3), turned to 120 degrees
- moved R23 289.9 mm to (245.8, 248.2), turned to -60 degrees
- moved C14 281.7 mm to (259.6, 112.5), turned to 30 degrees
- moved U17 280.8 mm to (277.4, 213.1), turned to -30 degrees
- moved C15 279.1 mm to (257.3, 106.4), turned to -150 degrees
- moved U16 277.4 mm to (246.4, 258.1), turned to -60 degrees
- moved C39 274.6 mm to (199.9, 282.3), turned to 90 degrees
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Connections:
- net Net-(SW1-A) renamed /Power & Voltage Regulators/SW_VCC
- C11 pad 1: Net-(U6-VBST) -> VCC
- C11 pad 2: Net-(U6-SW) -> GND
- C12 pad 1: VCC -> Net-(U6-VBST)
- C12 pad 2: GND -> Net-(U6-SW)
Routing:
- net +3.3V: track 0.00 -> 387.6 mm, vias 0 -> 20
- net +5V: track 0.00 -> 312.5 mm, vias 0 -> 5
- net GND: track 0.00 -> 87.3 mm, vias 0 -> 43
- net VCC: track 0.00 -> 65.2 mm, vias 0 -> 12
- net /Power & Voltage Regulators/SW_VCC: track 0.00 -> 33.0 mm
- net Net-(U16-VFB): track 0.00 -> 17.4 mm
- net Net-(U11-VFB): track 0.00 -> 17.0 mm
- net Net-(U6-VFB): track 0.00 -> 17.0 mm
- net Net-(U7-VFB): track 0.00 -> 16.9 mm
- net Net-(U14-VFB): track 0.00 -> 16.9 mm
- net Net-(U12-VFB): track 0.00 -> 16.9 mm
- net Net-(U15-VFB): track 0.00 -> 16.9 mm
- net Net-(U8-VFB): track 0.00 -> 16.9 mm
- net Net-(U13-VFB): track 0.00 -> 16.8 mm
- net Net-(U10-VFB): track 0.00 -> 16.8 mm
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- added copper zone on In1.Cu, net GND
- added copper zone on In2.Cu, net VCC
Other:
- board size 228.6 x 228.6 mm -> 226.6 x 226.6 mm
