File: development/arena_12-12_w_vreg/ni/ni_arena_12-12_v0p1/ni_arena_12-12_copy.kicad_pcb (KiCad board)
At the start: 4 copper layers, 228.6 x 228.6 mm, 126 parts, among them J1 Barrel_Jack, J2 NI_TE_68pos, P1 CONN15, P10 CONN15, P11 CONN15, P12 CONN15, P2 CONN15, P3 CONN15, P4 CONN15, P5 CONN15, P6 CONN15, P7 CONN15, P8 CONN15, P9 CONN15, Q2 MOSFET_NCHAN, SW1 SW_SPDT, U1 TXB0108PW, U10 TPS564201DDC, U11 TPS564201DDC, U12 TPS564201DDC, U13 TPS564201DDC, U14 TPS564201DDC, U15 TPS564201DDC, U16 TPS564201DDC, U17 TPS564201DDC, U18 AP2112K-3.3, U2 TXB0108PW, U3 TXB0108PW, U4 TXB0108PW, U5 TXB0108PW, U6 TPS564201DDC, U7 TPS564201DDC, U8 TPS564201DDC, U9 TPS564201DDC

Commit message: Worked on routing for ni and teensy vreg arenas.
Parts:
- C11: value 100nF -> 10uF
- C12: value 10uF -> 100nF
- moved C44 332.5 mm to (276.3, 206.2), turned to 60 degrees
- moved C45 326.2 mm to (271.5, 203.4), turned to -120 degrees
- moved C46 323.2 mm to (269.1, 204.0), turned to -120 degrees
- moved C41 321.3 mm to (249.0, 251.6), turned to 30 degrees
- moved C42 315.6 mm to (246.2, 246.8), turned to -150 degrees
- moved R26 312.1 mm to (267.4, 203.1), turned to -120 degrees
- moved C43 312.0 mm to (243.8, 246.1), turned to -150 degrees
- moved R25 310.9 mm to (265.6, 202.0), turned to 60 degrees
- moved R24 308.9 mm to (242.8, 244.5), turned to -150 degrees
- moved R23 308.4 mm to (241.8, 242.7), turned to 30 degrees
- moved U17 299.9 mm to (273.4, 205.8), turned to 60 degrees
- moved C38 298.8 mm to (202.5, 277.3)
- moved C14 298.5 mm to (251.6, 106.6), turned to 120 degrees
- moved L12 297.5 mm to (270.3, 210.7), turned to 150 degrees
- moved U16 297.4 mm to (246.6, 249.8), turned to 30 degrees
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Connections:
- net Net-(SW1-A) renamed /Power & Voltage Regulators/SW_VCC
- C11 pad 1: Net-(U6-VBST) -> VCC
- C11 pad 2: Net-(U6-SW) -> GND
- C12 pad 1: VCC -> Net-(U6-VBST)
- C12 pad 2: GND -> Net-(U6-SW)
- C47 pad 1: /Level Shifters/POW.5V_HDR_1 -> /Level Shifters/POW.5V_HDR_10
- U18 pad 1: /Level Shifters/POW.5V_HDR_1 -> /Level Shifters/POW.5V_HDR_10
- U18 pad 3: /Level Shifters/POW.5V_HDR_1 -> /Level Shifters/POW.5V_HDR_10
Routing:
- net /Level Shifters/POW.5V_HDR_10: track 0.00 -> 213.9 mm, vias 0 -> 7
- net +3.3V: track 0.00 -> 198.4 mm, vias 0 -> 11
- net GND: track 0.00 -> 136.0 mm, vias 0 -> 41
- net VCC: track 0.00 -> 73.6 mm, vias 0 -> 12
- net /Power & Voltage Regulators/SW_VCC: track 0.00 -> 31.5 mm
- net /Level Shifters/POW.5V_HDR_5: track 0.00 -> 15.7 mm
- net /Level Shifters/POW.5V_HDR_3: track 0.00 -> 15.6 mm
- net /Level Shifters/POW.5V_HDR_1: track 0.00 -> 15.5 mm
- net /Level Shifters/POW.5V_HDR_2: track 0.00 -> 15.3 mm
- net /Level Shifters/POW.5V_HDR_4: track 0.00 -> 15.2 mm
- net /Level Shifters/POW.5V_HDR_7: track 0.00 -> 15.2 mm
- net /Level Shifters/POW.5V_HDR_6: track 0.00 -> 15.1 mm
- net /Level Shifters/POW.5V_HDR_8: track 0.00 -> 15.1 mm
- net /Level Shifters/POW.5V_HDR_12: track 0.00 -> 15.0 mm
- net /Level Shifters/POW.5V_HDR_11: track 0.00 -> 14.9 mm
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- added copper zone on In1.Cu, net GND
- added copper zone on In2.Cu, net VCC
Other:
- board text added: "NI 12-12 VREG ARENA V0.1 R1"
- board text removed: "NI 12-12 Arena V0.1 R1"
