File: development/arena_12-12_w_vreg/ni/ni_arena_12-12_v0p1/power.kicad_sch (KiCad schematic)
At the start: 89 parts, among them J1 Barrel_Jack, SW1 SW_SPDT, U10 TPS564201DDC, U11 TPS564201DDC, U12 TPS564201DDC, U13 TPS564201DDC, U14 TPS564201DDC, U15 TPS564201DDC, U16 TPS564201DDC, U17 TPS564201DDC, U18 AP2112K-3.3, U6 TPS564201DDC, U7 TPS564201DDC, U8 TPS564201DDC, U9 TPS564201DDC

Commit message: Worked on routing for ni and teensy vreg arenas.
Parts:
- renumbered C12 to C11, C11 to C12
Connections:
- net SW_VCC: now reaches J1.1, SW1.1 (A)
Changed lines of the file:
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@@
     (effects (font (size 1.27 1.27)) (justify right bottom))
+  )
+  (label "SW_VCC" (at 47.371 213.233 0) (fields_autoplaced)
+    (effects (font (size 1.27 1.27)) (justify left bottom))
   )
   (label "POW.5V_HDR_3" (at 107.315 104.267 180) (fields_autoplaced)
@@
   (symbol (lib_id "Device:C_Small") (at 39.37 45.212 0) (unit 1)
     (in_bom yes) (on_board yes) (dnp no)
-    (property "Reference" "C12" (at 33.02 43.307 0)
+    (property "Reference" "C11" (at 33.02 43.307 0)
       (effects (font (size 1.27 1.27)) (justify left))
     )
@@
       (project "ni_arena_12-12"
         (path "/a2511654-3a17-43f1-8b9e-c45e375533dc/17861c68-32c3-4000-8a50-4f303c28fa47"
-          (reference "C12") (unit 1)
+          (reference "C11") (unit 1)
         )
       )
@@
   (symbol (lib_id "Device:C_Small") (at 64.77 37.592 180) (unit 1)
     (in_bom yes) (on_board yes) (dnp no)
-    (property "Reference" "C11" (at 71.12 36.322 0)
+    (property "Reference" "C12" (at 71.12 36.322 0)
       (effects (font (size 1.27 1.27)) (justify left))
     )
@@
       (project "ni_arena_12-12"
         (path "/a2511654-3a17-43f1-8b9e-c45e375533dc/17861c68-32c3-4000-8a50-4f303c28fa47"
-          (reference "C11") (unit 1)
-        )
-      )
+          (reference "C12") (unit 1)
+        )
+      )
