File: development/arena_12-12_w_vreg/ni/ni_arena_12-12_v0p1/ni_connector.kicad_sch (KiCad schematic)
At the start: 1 part, among them J2 NI_TE_68pos

Commit message: Work on BOMs for 12-12 arenas with vregs. Finish non-LSCS versions.
Other:
- note added: "68-pin DSUB for NI cable, vertical TE Connectivity 5174339-5 Digikey PN A123166-ND"
- note removed: "68-pin DSUB for NI cable RA TE Connectivity 2-5174225-5 Digikey PN A33476-ND Vertical TE Connectivity Digikey"
Changed lines of the file:
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@@
     (stroke (width 0) (type default))
   )
-  (text "68-pin DSUB for NI cable  \n\nRA\nTE Connectivity 2-5174225-5\nDigikey PN A33476-ND\n\nVertical\nTE Connectivity \nDigikey "
+  (text "68-pin DSUB for NI cable, vertical\nTE Connectivity 5174339-5\nDigikey PN A123166-ND\n\n"
     (at 74.93 177.038 0)
     (effects (font (size 2.032 2.032)) (justify left bottom))
