File: development/arena_12-12_w_vreg/ni/ni_arena_12-12_v0p1/layout_tool/modified_ni_arena_12-12.kicad_pcb (KiCad board)
At the start: 4 copper layers, 228.6 x 228.6 mm, 126 parts, among them J1 Barrel_Jack, J2 NI_TE_68pos, P1 CONN15, P10 CONN15, P11 CONN15, P12 CONN15, P2 CONN15, P3 CONN15, P4 CONN15, P5 CONN15, P6 CONN15, P7 CONN15, P8 CONN15, P9 CONN15, Q2 MOSFET_NCHAN, SW1 SW_SPDT, U1 TXB0108PW, U10 TPS564201DDC, U11 TPS564201DDC, U12 TPS564201DDC, U13 TPS564201DDC, U14 TPS564201DDC, U15 TPS564201DDC, U16 TPS564201DDC, U17 TPS564201DDC, U18 AP2112K-3.3, U2 TXB0108PW, U3 TXB0108PW, U4 TXB0108PW, U5 TXB0108PW, U6 TPS564201DDC, U7 TPS564201DDC, U8 TPS564201DDC, U9 TPS564201DDC

Commit message: Worked on routing for ni and teensy vreg arenas.
Parts:
- C11: value 100nF -> 10uF
- C12: value 10uF -> 100nF
- moved C48 35.2 mm to (186.9, 283.9), turned to -90 degrees
- moved U18 30.9 mm to (189.9, 284.1), turned to 90 degrees
- moved C47 30.2 mm to (191.2, 287.5), turned to 180 degrees
- moved U3 15.0 mm to (229.8, 285.4)
- moved C5 15.0 mm to (235.9, 287.7)
- moved C6 15.0 mm to (223.4, 287.7)
- moved C3 14.9 mm to (129.8, 287.7)
- moved U2 14.9 mm to (123.8, 285.4)
- moved C4 14.9 mm to (117.5, 287.7)
- moved C14 8.96 mm to (251.6, 106.6), turned to 120 degrees
- moved C23 8.96 mm to (106.6, 104.0), turned to -150 degrees
- moved C32 8.96 mm to (104.0, 249.0), turned to -60 degrees
- moved C41 8.96 mm to (249.0, 251.6), turned to 30 degrees
- moved C38 8.96 mm to (202.5, 277.3), turned to 0 degrees
- moved C17 8.96 mm to (206.2, 79.3), turned to 150 degrees
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Connections:
- net Net-(SW1-A) renamed /Power & Voltage Regulators/SW_VCC
- C11 pad 1: Net-(U6-VBST) -> VCC
- C11 pad 2: Net-(U6-SW) -> GND
- C12 pad 1: VCC -> Net-(U6-VBST)
- C12 pad 2: GND -> Net-(U6-SW)
- C47 pad 1: /Level Shifters/POW.5V_HDR_1 -> /Level Shifters/POW.5V_HDR_10
- U18 pad 1: /Level Shifters/POW.5V_HDR_1 -> /Level Shifters/POW.5V_HDR_10
- U18 pad 3: /Level Shifters/POW.5V_HDR_1 -> /Level Shifters/POW.5V_HDR_10
Routing:
- net /Power & Voltage Regulators/SW_VCC: track 0.00 -> 31.5 mm
- net /Level Shifters/POW.5V_HDR_1: track 0.00 -> 15.5 mm
- net GND: track 0.00 -> 13.4 mm, vias 0 -> 3
- net Net-(U6-VFB): track 0.00 -> 12.6 mm
- net Net-(U6-SW): track 0.00 -> 10.6 mm
- net VCC: track 0.00 -> 6.11 mm, vias 0 -> 1
- net Net-(Q2-G): track 0.00 -> 5.19 mm
- net Net-(U6-VBST): track 0.00 -> 2.12 mm
- added copper zone on In1.Cu, net GND
- added copper zone on In2.Cu, net VCC
Other:
- board text added: "NI 12-12 VREG ARENA V0.1 R1"
- board text removed: "NI 12-12 Arena V0.1 R1"
