File: development/arena_12-12/teensy4p1/teensy_arena_12-12_v0p1/teensy_arena_12-12_tmp.kicad_pcb (KiCad board)
At the start: 4 copper layers, 254 x 254 mm, 87 parts, among them J1 Barrel_Jack, J2 Conn_01x04, J3 Conn_01x04, P1 CONN15, P10 CONN15, P11 CONN15, P12 CONN15, P2 CONN15, P3 CONN15, P4 CONN15, P5 CONN15, P6 CONN15, P7 CONN15, P8 CONN15, P9 CONN15, Q2 MOSFET_NCHAN, SW1 SW_SPDT, U1 TXB0108PW, U10 AZ1084-5.0, U11 AZ1084-5.0, U12 AZ1084-5.0, U13 AZ1084-5.0, U14 AZ1084-5.0, U15 AZ1084-5.0, U16 AZ1084-5.0, U17 AZ1084-5.0, U18 Teensy4.1, U2 TXB0108PW, U3 TXB0108PW, U4 TXB0108PW, U5 TXB0108PW, U6 AZ1084-5.0, U7 AZ1084-5.0, U8 AZ1084-5.0, U9 AZ1084-5.0

Commit message: Added routing of teensy 12-12 arena with big caps.
Parts:
- removed C23, C25, C27, C29, C31, C33: 10uF, Capacitor_SMD:CP_Elec_4x5.4
- removed C24, C26, C28, C30, C32, C34: 22uF, Capacitor_SMD:CP_Elec_4x5.4
- removed R10, R11, R12, R13, R14, R3, R4, R5, R6, R7, R8, R9: 300, Capacitor_SMD:C_1206_3216Metric
- removed U10, U11, U12, U13, U14, U15, U16, U17, U6, U7, U8, U9: AZ1084-5.0, Package_TO_SOT_SMD:TO-252-3_TabPin2
- C11, C13, C15, C17, C21: value 10uF -> 100uF; footprint Capacitor_SMD:CP_Elec_4x5.4 -> Capacitor_SMD:C_1210_3225Metric
- C12, C14, C16, C18, C20, C22: value 22uF -> 100uF; footprint Capacitor_SMD:CP_Elec_4x5.4 -> Capacitor_SMD:C_1210_3225Metric
- C19: value 10F -> 100uF; footprint Capacitor_SMD:CP_Elec_4x5.4 -> Capacitor_SMD:C_1210_3225Metric
- J2, J3: footprint Connector_JST:JST_SH_SM04B-SRSS-TB_1x04-1MP_P1.00mm_Horizontal -> arena_custom:JST_SH_SM04B-SRSS-TB_1x04-1MP_P1.00mm_Horizontal
- moved C21 200.2 mm to (239.8, 251.8), turned to -150 degrees
- moved C20 196.7 mm to (194.5, 272.9), turned to 180 degrees
- moved C22 196.0 mm to (268.5, 210.9), turned to -120 degrees
- moved C19 190.6 mm to (144.7, 268.5), turned to 150 degrees
- moved C18 183.9 mm to (103.8, 239.8), turned to 120 degrees
- moved C17 168.0 mm to (82.7, 194.5)
- moved C16 158.7 mm to (87.1, 144.7), turned to 60 degrees
- moved C15 134.0 mm to (115.8, 103.8), turned to 30 degrees
- moved C14 122.6 mm to (161.1, 82.7), turned to 0 degrees
- moved C8 108.0 mm to (154.1, 286.4)
- moved U4 107.9 mm to (160.3, 284.1)
- moved C7 107.8 mm to (166.8, 286.3)
- moved C13 91.0 mm to (210.9, 87.1), turned to -30 degrees
- moved C12 78.2 mm to (251.8, 115.8), turned to -60 degrees
- moved J2 78.2 mm to (288.7, 162.4)
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Connections:
- net Net-(SW1-A) renamed /Power/SW_5V
- C11 pad 1: VCC -> +5V
- C12 pad 1: /Panel Headers/POW.5V_HDR_1 -> +5V
- C13 pad 1: VCC -> +5V
- C14 pad 1: /Panel Headers/POW.5V_HDR_2 -> +5V
- C15 pad 1: VCC -> +5V
- C16 pad 1: /Panel Headers/POW.5V_HDR_3 -> +5V
- C17 pad 1: VCC -> +5V
- C18 pad 1: /Panel Headers/POW.5V_HDR_4 -> +5V
- C19 pad 1: VCC -> +5V
- C20 pad 1: /Panel Headers/POW.5V_HDR_5 -> +5V
- C21 pad 1: VCC -> +5V
- C22 pad 1: /Panel Headers/POW.5V_HDR_6 -> +5V
- P1 pad 1: /Panel Headers/POW.5V_HDR_1 -> +5V
- P1 pad 3: /Level Shifters/PAN5V.SCK_1 -> /Panel Headers/RESET
- P10 pad 1: /Panel Headers/POW.5V_HDR_10 -> +5V
- P10 pad 3: /Level Shifters/PAN5V.SCK_1 -> /Panel Headers/RESET
- P11 pad 1: /Panel Headers/POW.5V_HDR_11 -> +5V
- P11 pad 3: /Level Shifters/PAN5V.SCK_1 -> /Panel Headers/RESET
- P12 pad 1: /Panel Headers/POW.5V_HDR_12 -> +5V
- P12 pad 3: /Level Shifters/PAN5V.SCK_1 -> /Panel Headers/RESET
- P2 pad 1: /Panel Headers/POW.5V_HDR_2 -> +5V
- P2 pad 3: /Level Shifters/PAN5V.SCK_1 -> /Panel Headers/RESET
- P2 pad 9: /Level Shifters/PAN5V.CS_06 -> /Level Shifters/PAN5V.CS_07
- P3 pad 1: /Panel Headers/POW.5V_HDR_3 -> +5V
- P3 pad 3: /Level Shifters/PAN5V.SCK_1 -> /Panel Headers/RESET
- P4 pad 1: /Panel Headers/POW.5V_HDR_4 -> +5V
- P4 pad 3: /Level Shifters/PAN5V.SCK_1 -> /Panel Headers/RESET
- P5 pad 1: /Panel Headers/POW.5V_HDR_5 -> +5V
- P5 pad 3: /Level Shifters/PAN5V.SCK_1 -> /Panel Headers/RESET
- P6 pad 1: /Panel Headers/POW.5V_HDR_6 -> +5V
- P6 pad 3: /Level Shifters/PAN5V.SCK_1 -> /Panel Headers/RESET
- P7 pad 1: /Panel Headers/POW.5V_HDR_7 -> +5V
- P7 pad 3: /Level Shifters/PAN5V.SCK_1 -> /Panel Headers/RESET
- P8 pad 1: /Panel Headers/POW.5V_HDR_8 -> +5V
- P8 pad 3: /Level Shifters/PAN5V.SCK_1 -> /Panel Headers/RESET
- P8 pad 9: /Level Shifters/PAN5V.CS_06 -> /Level Shifters/PAN5V.CS_07
- P9 pad 1: /Panel Headers/POW.5V_HDR_9 -> +5V
- P9 pad 3: /Level Shifters/PAN5V.SCK_1 -> /Panel Headers/RESET
- Q2 pad 3: /Level Shifters/PAN5V.SCK_1 -> /Panel Headers/RESET
- SW1 pad 2: VCC -> +5V
- U18 pad 48: +5V -> unconnected-(U18-VIN-Pad48)
- U18 pad 49: +5V -> unconnected-(U18-VUSB-Pad49)
Routing:
- net VCC: track 1078.7 -> 0.00 mm, vias 12 -> 0
- net /Panel Headers/RESET: track 0.00 -> 613.6 mm, vias 0 -> 8
- net /Level Shifters/PAN5V.CS_07: track 0.00 -> 332.9 mm, vias 0 -> 2
- net /Level Shifters/PAN5V.SCK_1: track 619.6 -> 306.0 mm, vias 1 -> 3
- net GND: track 346.1 -> 97.4 mm, vias 42 -> 13
- net +5V: track 237.8 -> 90.9 mm
- net +3.3V: track 289.8 -> 394.0 mm, vias 11 -> 12
- net /Level Shifters/PAN3V.CS_19: track 25.8 -> 128.4 mm, vias 0 -> 2
- net /Level Shifters/PAN5V.CS_19: track 399.6 -> 301.3 mm, vias 1 -> 5
- net /Level Shifters/PAN3V.CS_21: track 18.7 -> 116.6 mm, vias 0 -> 3
- net /Level Shifters/PAN3V.CS_17: track 31.4 -> 128.4 mm, vias 0 -> 1
- net /Level Shifters/PAN3V.CS_18: track 28.6 -> 125.3 mm
- net /Level Shifters/PAN3V.CS_20: track 22.9 -> 118.6 mm
- net /Level Shifters/PAN3V.CS_22: track 16.9 -> 111.7 mm, vias 0 -> 2
- net /Level Shifters/PAN3V.CS_23: track 15.8 -> 102.7 mm, vias 0 -> 2
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- added copper zone on In2.Cu, net +5V
- removed copper zone on In2.Cu, net GND
Other:
- board size 254 x 254 mm -> 228.6 x 228.6 mm
- board text added: "3.3V"
- board text added: "5V"
- board text added: "A0"
- board text added: "A1"
- board text added: "ANALOG IN"
- board text added: "GND"
- board text added: "ON OFF"
- board text added: "QWIIC/QT"
- board text added: "SCL"
- board text added: "SDA"
- board text added: "Teensy 12-12 Controller-Arena V0.1 R1"
