File: development/arena_12-12_w_vreg/ni/ni_arena_12-12_v0p1/copies/ni_arena_12-12_partial_route_for_fix.kicad_pcb (KiCad board)
At the start: 6 copper layers, 228.6 x 228.6 mm, 126 parts, among them J1 Barrel_Jack, J2 NI_TE_68pos, P1 CONN15, P10 CONN15, P11 CONN15, P12 CONN15, P2 CONN15, P3 CONN15, P4 CONN15, P5 CONN15, P6 CONN15, P7 CONN15, P8 CONN15, P9 CONN15, Q2 MOSFET_NCHAN, SW1 SW_SPDT, U1 TXB0108PW, U10 TPS564201DDC, U11 TPS564201DDC, U12 TPS564201DDC, U13 TPS564201DDC, U14 TPS564201DDC, U15 TPS564201DDC, U16 TPS564201DDC, U17 TPS564201DDC, U18 AP2112K-3.3, U2 TXB0108PW, U3 TXB0108PW, U4 TXB0108PW, U5 TXB0108PW, U6 TPS564201DDC, U7 TPS564201DDC, U8 TPS564201DDC, U9 TPS564201DDC

Commit message: Intermediate save during re-route of NI 12-12 arena with vreg.
Parts:
- turned J2 to 90 degrees
Routing:
- net /Level Shifters/PAN5V.CS_03: track 0.00 -> 620.4 mm, vias 0 -> 6
- net /Level Shifters/PAN5V.CS_06: track 0.00 -> 618.2 mm, vias 0 -> 7
- net /Level Shifters/PAN5V.CS_05: track 0.00 -> 615.4 mm, vias 0 -> 8
- net /Level Shifters/PAN5V.CS_02: track 0.00 -> 613.1 mm, vias 0 -> 5
- net /Level Shifters/PAN5V.CS_04: track 0.00 -> 610.0 mm, vias 0 -> 8
- net /Level Shifters/PAN5V.CS_01: track 13.8 -> 623.8 mm, vias 1 -> 6
- net /Level Shifters/PAN5V.CS_00: track 0.00 -> 607.8 mm, vias 0 -> 9
- net /Level Shifters/PAN5V.CS_07: track 0.00 -> 605.3 mm, vias 0 -> 5
- net /Panel Headers/RESET: track 0.00 -> 589.4 mm, vias 0 -> 4
- net /Level Shifters/PAN5V.EXT_INT: track 0.00 -> 576.5 mm, vias 0 -> 6
- net /Level Shifters/PAN5V.SCK_00: track 0.00 -> 337.4 mm, vias 0 -> 5
- net /Level Shifters/PAN5V.SCK_02: track 0.00 -> 336.8 mm, vias 0 -> 4
- net /Level Shifters/PAN5V.SCK_01: track 0.00 -> 333.5 mm, vias 0 -> 3
- net /Level Shifters/PAN5V.SCK_04: track 0.00 -> 331.6 mm, vias 0 -> 3
- net /Level Shifters/PAN5V.SCK_05: track 0.00 -> 329.6 mm, vias 0 -> 5
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