File: legacy/other_older_designs/arena_6-inf_v0p3/arena_6-inf_v0p3.kicad_sch (KiCad schematic)
At the start: 34 parts, among them J1 Conn_02x34_Counter_Clockwise, J2 Conn_02x34_Top_Bottom, P1 CONN15, P10 CONN_20X2, P2 CONN15, P3 CONN15, P4 CONN15, P5 CONN15, P6 CONN15, P7 CONN_20X2, P9 CONN_2, Q1 MOSFET_NCHAN, SW1 SWITCH_INV, U1 SPARKFUN_TXB0104, U2 SPARKFUN_TXB0104, U3 SPARKFUN_TXB0104, U4 SPARKFUN_TXB0104, U5 SPARKFUN_TXB0104, U6 SPARKFUN_TXB0104, U7 SPARKFUN_TXB0104, U8 POLOLU_3V3

Commit message: Fix issue on legacy design.
Parts:
- removed J1: Conn_02x34_Counter_Clockwise, symbol Connector_Generic:Conn_02x34_Counter_Clockwise
